Commit message: update model
update model and urdf

File: elfin15/elfin15_ros2_gazebo/urdf/elfin15.urdf.xacro (robot description, xacro)
@@ -30,5 +30,5 @@
     <origin
       xyz="0 0 0"
-      rpy="0 0 1.5708" />
+      rpy="0 0 0" />
     <parent
       link="elfin_base_link" />
@@ -40,15 +40,15 @@
     <inertial>
       <origin
-        xyz="2.654E-09 0.0003357 0.036153"
-        rpy="0 0 0" />
-      <mass
-        value="2.8356" />
-      <inertia
-        ixx="0.0097381"
-        ixy="-1.8821E-10"
-        ixz="-9.0965E-11"
-        iyy="0.0098176"
-        iyz="2.182E-05"
-        izz="0.016617" />
+        xyz="-0.00136943117439078 -2.2883687794971E-06 0.037653456901999"
+        rpy="0 0 0" />
+      <mass
+        value="7.29685766810245" />
+      <inertia
+        ixx="0.0253289354355793"
+        ixy="9.31156473219125E-08"
+        ixz="-0.000185995712246883"
+        iyy="0.0242633188941406"
+        iyz="-5.25886087064228E-07"
+        izz="0.0424125697382868" />
     </inertial>
     <visual>
@@ -63,5 +63,5 @@
         name="">
         <color
-          rgba="0.86667 0.86667 0.8902 1" />
+          rgba="0.866666666666667 0.866666666666667 0.890196078431372 1" />
       </material>
     </visual>
@@ -80,15 +80,15 @@
     <inertial>
       <origin
-        xyz="-0.0040174 0.2265 4.5331E-06"
-        rpy="0 0 0" />
-      <mass
-        value="9.7894" />
-      <inertia
-        ixx="0.07916"
-        ixy="0.0021604"
-        ixz="4.5316E-06"
-        iyy="0.060146"
-        iyz="-5.7743E-06"
-        izz="0.088867" />
+        xyz="-1.88838434646975E-06 -0.00357534605111417 -0.0358732421913592"
+        rpy="0 0 0" />
+      <mass
+        value="26.1752707800957" />
+      <inertia
+        ixx="0.235852905806904"
+        ixy="-2.93045226725672E-06"
+        ixz="-7.40247338756675E-06"
+        iyy="0.211816347359602"
+        iyz="0.00543673722583904"
+        izz="0.158448663526753" />
     </inertial>
     <visual>
@@ -103,5 +103,5 @@
         name="">
         <color
-          rgba="0.79216 0.81961 0.93333 1" />
+          rgba="1 1 1 1" />
       </material>
     </visual>
@@ -118,4 +118,62 @@
   <joint
     name="elfin_joint1"
+    type="revolute">
+    <origin
+      xyz="0 0 0.262"
+      rpy="0 0 0" />
+    <parent
+      link="elfin_base" />
+    <child
+      link="elfin_link1" />
+    <axis
+      xyz="0 0 1" />
+    <limit
+      lower="-3.14"
+      upper="3.14"
+      effort="104"
+      velocity="1.57" />
+  </joint>
+  <link
+    name="elfin_link2">
+    <inertial>
+      <origin
+        xyz="2.05933361594049E-05 0.292081364859745 0.154041796903471"
+        rpy="0 0 0" />
+      <mass
+        value="25.7826523644554" />
+      <inertia
+        ixx="1.59115969876519"
+        ixy="-0.000158434707227747"
+        ixz="-1.28374843136211E-05"
+        iyy="0.060560052287277"
+        iyz="0.0849224026877452"
+        izz="1.60940122192142" />
+    </inertial>
+    <visual>
+      <origin
+        xyz="0 0 0"
+        rpy="0 0 0" />
+      <geometry>
+        <mesh
+          filename="file://$(find elfin_description)/meshes/elfin15/elfin_link2.STL" />
+      </geometry>
+      <material
+        name="">
+        <color
+          rgba="0.890196078431372 0.890196078431372 0.913725490196078 1" />
+      </material>
+    </visual>
+    <collision>
+      <origin
+        xyz="0 0 0"
+        rpy="0 0 0" />
+      <geometry>
+        <mesh
+          filename="file://$(find elfin_description)/meshes/elfin15/elfin_link2.STL" />
+      </geometry>
+    </collision>
+  </link>
+  <joint
+    name="elfin_joint2"
     type="revolute">
     <origin
@@ -123,72 +181,14 @@
       rpy="1.5708 0 0" />
     <parent
-      link="elfin_base" />
-    <child
       link="elfin_link1" />
-    <axis
-      xyz="0 1 0" />
-    <limit
-      lower="-3.14"
-      upper="3.14"
-      effort="420"
-      velocity="1.57" />
-  </joint>
-  <link
-    name="elfin_link2">
-    <inertial>
-      <origin
-        xyz="-0.035073 0.29215 1.7591E-05"
-        rpy="0 0 0" />
-      <mass
-        value="9.5865" />
-      <inertia
-        ixx="0.59803"
-        ixy="-0.031615"
-        ixz="4.8599E-06"
-        iyy="0.022645"
-        iyz="-4.8185E-05"
-        izz="0.59118" />
-    </inertial>
-    <visual>
-      <origin
-        xyz="0 0 0"
-        rpy="0 0 0" />
-      <geometry>
-        <mesh
-          filename="file://$(find elfin_description)/meshes/elfin15/elfin_link2.STL" />
-      </geometry>
-      <material
-        name="">
-        <color
-          rgba="0.8902 0.8902 0.9098 1" />
-      </material>
-    </visual>
-    <collision>
-      <origin
-        xyz="0 0 0"
-        rpy="0 0 0" />
-      <geometry>
-        <mesh
-          filename="file://$(find elfin_description)/meshes/elfin15/elfin_link2.STL" />
-      </geometry>
-    </collision>
-  </link>
-  <joint
-    name="elfin_joint2"
-    type="revolute">
-    <origin
-      xyz="-0.121 0.262 0"
-      rpy="0 0 0" />
-    <parent
-      link="elfin_link1" />
     <child
       link="elfin_link2" />
     <axis
-      xyz="-1 0 0" />
+      xyz="0 0 1" />
     <limit
       lower="-2.35"
       upper="2.35"
-      effort="420"
-      velocity="1.57" />
+      effort="104"
+      velocity="1.27" />
   </joint>
   <link
@@ -196,15 +196,15 @@
     <inertial>
       <origin
-        xyz="-0.0049696 -0.035269 2.0786E-06"
-        rpy="0 0 0" />
-      <mass
-        value="2.9386" />
-      <inertia
-        ixx="0.011876"
-        ixy="0.00059921"
-        ixz="1.0886E-07"
-        iyy="0.0075913"
-        iyz="4.8168E-07"
-        izz="0.013762" />
+        xyz="0.0361013116039101 -2.09104451848553E-06 -0.00436986898383294"
+        rpy="0 0 0" />
+      <mass
+        value="7.87585395095179" />
+      <inertia
+        ixx="0.0200598769348272"
+        ixy="1.25572941880986E-06"
+        ixz="-0.00144896285503519"
+        iyy="0.0366449882644546"
+        iyz="-3.00644865145763E-07"
+        izz="0.0318875682141342" />
     </inertial>
     <visual>
@@ -236,6 +236,6 @@
     type="revolute">
     <origin
-      xyz="0.121 0.73 0"
-      rpy="3.1416 0 0" />
+      xyz="0 0.73 0"
+      rpy="3.1416 0 1.5708" />
     <parent
       link="elfin_link2" />
@@ -243,179 +243,63 @@
       link="elfin_link3" />
     <axis
-      xyz="1 0 0" />
+      xyz="0 0 1" />
     <limit
       lower="-2.61"
       upper="2.61"
-      effort="200"
-      velocity="1.57" />
-  </joint>
-  <link
-    name="elfin_link4">
-    <inertial>
-      <origin
-        xyz="-0.064982 0.17333 3.5794E-05"
-        rpy="0 0 0" />
-      <mass
-        value="2.8258" />
-      <inertia
-        ixx="0.055923"
-        ixy="0.01272"
-        ixz="3.6239E-06"
-        iyy="0.0079448"
-        iyz="-1.9213E-05"
-        izz="0.060085" />
-    </inertial>
-    <visual>
-      <origin
-        xyz="0 0 0"
-        rpy="0 0 0" />
-      <geometry>
-        <mesh
-          filename="file://$(find elfin_description)/meshes/elfin15/elfin_link4.STL" />
-      </geometry>
-      <material
-        name="">
-        <color
-          rgba="0.79216 0.81961 0.93333 1" />
-      </material>
-    </visual>
-    <collision>
-      <origin
-        xyz="0 0 0"
-        rpy="0 0 0" />
-      <geometry>
-        <mesh
-          filename="file://$(find elfin_description)/meshes/elfin15/elfin_link4.STL" />
-      </geometry>
-    </collision>
-  </link>
-  <joint
-    name="elfin_joint4"
-    type="revolute">
-    <origin
-      xyz="0 -0.147 0"
-      rpy="-3.1416 0 0" />
-    <parent
-      link="elfin_link3" />
-    <child
-      link="elfin_link4" />
-    <axis
-      xyz="0 1 0" />
-    <limit
-      lower="-3.14"
-      upper="3.14"
-      effort="200"
-      velocity="1.57" />
-  </joint>
-  <link
-    name="elfin_link5">
-    <inertial>
-      <origin
-        xyz="-0.002491 -0.025023 -6.7752E-06"
-        rpy="0 0 0" />
-      <mass
-        value="1.2566" />
-      <inertia
-        ixx="0.0027306"
-        ixy="9.9756E-05"
-        ixz="4.9287E-07"
-        iyy="0.0020256"
-        iyz="-2.707E-07"
-        izz="0.0034996" />
-    </inertial>
-    <visual>
-      <origin
-        xyz="0 0 0"
-        rpy="0 0 0" />
-      <geometry>
-        <mesh
-          filename="file://$(find elfin_description)/meshes/elfin15/elfin_link5.STL" />
-      </geometry>
-      <material
-        name="">
-        <color
-          rgba="0.8902 0.8902 0.9098 1" />
-      </material>
-    </visual>
-    <collision>
-      <origin
-        xyz="0 0 0"
-        rpy="0 0 0" />
-      <geometry>
-        <mesh
-          filename="file://$(find elfin_description)/meshes/elfin15/elfin_link5.STL" />
-      </geometry>
-    </collision>
-  </link>
-  <joint
-    name="elfin_joint5"
-    type="revolute">
-    <origin
-      xyz="0 0.42047 0"
-      rpy="3.1416 0 0" />
-    <parent
-      link="elfin_link4" />
-    <child
-      link="elfin_link5" />
-    <axis
-      xyz="1 0 0" />
-    <limit
-      lower="-2.56"
-      upper="2.56"
       effort="69"
       velocity="1.57" />
   </joint>
   <link
-    name="elfin_link6">
-    <inertial>
-      <origin
-        xyz="-0.004035 -0.019415 1.3786E-07"
-        rpy="0 0 0" />
-      <mass
-        value="0.35802" />
-      <inertia
-        ixx="0.00025128"
-        ixy="4.2989E-06"
-        ixz="-3.5119E-11"
-        iyy="0.00035947"
-        iyz="-8.6185E-11"
-        izz="0.0002947" />
-    </inertial>
-    <visual>
-      <origin
-        xyz="0 0 0"
-        rpy="0 0 0" />
-      <geometry>
-        <mesh
-          filename="file://$(find elfin_description)/meshes/elfin15/elfin_link6.STL" />
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
File: elfin3/elfin3_ros2_gazebo/urdf/elfin3.urdf.xacro (robot description, xacro)
@@ -40,37 +40,37 @@
     <inertial>
       <origin
-        xyz="0.00425937844813294 -0.000389571231902992 0.00274262778667868"
-        rpy="0 0 0" />
-      <mass
-        value="0.0268461773395224" />
-      <inertia
-        ixx="2.66341322206443E-05"
-        ixy="5.51640996553045E-08"
-        ixz="2.21112209410463E-12"
-        iyy="2.67121402645769E-05"
-        iyz="-3.17722287525956E-12"
-        izz="5.30011200382481E-05" />
-    </inertial>
-    <visual>
-      <origin
-        xyz="0 0 0"
-        rpy="0 0 0" />
-      <geometry>
-        <mesh
-          filename="file://$(find elfin_description)/meshes/elfin3/base_link.STL" />
-      </geometry>
-      <material
-        name="">
-        <color
-          rgba="0.686274509803922 0.686274509803922 0.686274509803922 1" />
-      </material>
-    </visual>
-    <collision>
-      <origin
-        xyz="0 0 0"
-        rpy="0 0 0" />
-      <geometry>
-        <mesh
-          filename="file://$(find elfin_description)/meshes/elfin3/base_link.STL" />
+        xyz="-3.29424604565274E-17 -1.34268095035506E-13 0.0281618442441758"
+        rpy="0 0 0" />
+      <mass
+        value="0.957790548974336" />
+      <inertia
+        ixx="0.00150277910425554"
+        ixy="-5.07476794726385E-15"
+        ixz="6.74486887384113E-19"
+        iyy="0.00150277910426632"
+        iyz="-6.77700047631768E-15"
+        izz="0.00236857924691092" />
+    </inertial>
+    <visual>
+      <origin
+        xyz="0 0 0"
+        rpy="0 0 0" />
+      <geometry>
+        <mesh
+          filename="file://$(find elfin_description)/meshes/elfin3/elfin_base.STL" />
+      </geometry>
+      <material
+        name="">
+        <color
+          rgba="0.866666666666667 0.866666666666667 0.890196078431372 1" />
+      </material>
+    </visual>
+    <collision>
+      <origin
+        xyz="0 0 0"
+        rpy="0 0 0" />
+      <geometry>
+        <mesh
+          filename="file://$(find elfin_description)/meshes/elfin3/elfin_base.STL" />
       </geometry>
     </collision>
@@ -80,15 +80,15 @@
     <inertial>
       <origin
-        xyz="-1.11474311817293E-05 -0.019295238440266 0.081643413279284"
-        rpy="0 0 0" />
-      <mass
-        value="1.52628719338585" />
-      <inertia
-        ixx="0.006028902112623"
-        ixy="-5.48816506919481E-07"
-        ixz="-2.73302311360408E-07"
-        iyy="0.00509895338088794"
-        iyz="0.00146640275062038"
-        izz="0.0028687934642813" />
+        xyz="-9.91151833157951E-06 -0.00381802038981039 -0.0288793541460785"
+        rpy="0 0 0" />
+      <mass
+        value="1.76831994028414" />
+      <inertia
+        ixx="0.00611258909183611"
+        ixy="-9.83139510435094E-07"
+        ixz="-4.14810998305304E-07"
+        iyy="0.00490858433987136"
+        iyz="0.000238616259770754"
+        izz="0.00347391582535924" />
     </inertial>
     <visual>
@@ -103,5 +103,5 @@
         name="">
         <color
-          rgba="0.772549019607843 0.752941176470588 0.733333333333333 1" />
+          rgba="1 1 1 1" />
       </material>
     </visual>
@@ -120,5 +120,5 @@
     type="revolute">
     <origin
-      xyz="0 0 0.0695"
+      xyz="0 0 0.1925"
       rpy="0 0 0" />
     <parent
@@ -138,15 +138,15 @@
     <inertial>
       <origin
-        xyz="-3.09813419838078E-05 -0.0392725728395098 0.121906520746464"
-        rpy="0 0 0" />
-      <mass
-        value="0.519379765009091" />
-      <inertia
-        ixx="0.00462941997584524"
-        ixy="9.53033193206284E-08"
-        ixz="1.89958745191593E-06"
-        iyy="0.00485416387879526"
-        iyz="-0.00019166604937554"
-        izz="0.000506978474454832" />
+        xyz="-1.09591115591905E-05 0.119133426891285 0.104133324863746"
+        rpy="0 0 0" />
+      <mass
+        value="1.41431338277405" />
+      <inertia
+        ixx="0.015779563515351"
+        ixy="2.57229005873321E-06"
+        ixz="-1.33122516224454E-07"
+        iyy="0.00107744893104323"
+        iyz="0.000788193806414118"
+        izz="0.016037242338571" />
     </inertial>
     <visual>
@@ -161,5 +161,5 @@
         name="">
         <color
-          rgba="0.501960784313725 0.501960784313725 0.501960784313725 1" />
+          rgba="0.752941176470588 0.752941176470588 0.752941176470588 1" />
       </material>
     </visual>
@@ -178,6 +178,6 @@
     type="revolute">
     <origin
-      xyz="0 -0.066 0.123"
-      rpy="0 0 0" />
+      xyz="0 0 0"
+      rpy="1.5708 0 0" />
     <parent
       link="elfin_link1" />
@@ -185,5 +185,5 @@
       link="elfin_link2" />
     <axis
-      xyz="0 -1 0" />
+      xyz="0 0 1" />
     <limit
       lower="-2.35"
@@ -196,15 +196,15 @@
     <inertial>
       <origin
-        xyz="7.94789705792241E-06 0.0434911461385148 0.0377663456053925"
-        rpy="0 0 0" />
-      <mass
-        value="1.07924103107593" />
-      <inertia
-        ixx="0.00347290093864989"
-        ixy="-5.5219540256932E-07"
-        ixz="-1.81596933237452E-07"
-        iyy="0.0028883932232078"
-        iyz="-0.000859331225721596"
-        izz="0.00165138765596417" />
+        xyz="0.0250568861242891 6.90447572674757E-06 -0.00212484357202786"
+        rpy="0 0 0" />
+      <mass
+        value="1.24814802120785" />
+      <inertia
+        ixx="0.00198810458497945"
+        ixy="-2.27641402661824E-07"
+        ixz="-8.7904200299055E-05"
+        iyy="0.00344858240749365"
+        iyz="-4.73997143171874E-07"
+        izz="0.00270707588537784" />
     </inertial>
     <visual>
@@ -236,6 +236,6 @@
     type="revolute">
     <origin
-      xyz="0 0.005 0.266"
-      rpy="0 0 0" />
+      xyz="0 0.266 0"
+      rpy="3.1416 0 1.5708" />
     <parent
       link="elfin_link2" />
@@ -243,5 +243,5 @@
       link="elfin_link3" />
     <axis
-      xyz="0 1 0" />
+      xyz="0 0 1" />
     <limit
       lower="-2.61"
@@ -254,15 +254,15 @@
     <inertial>
       <origin
-        xyz="3.93948157579129E-06 -0.0583766984632963 0.104324949772583"
-        rpy="0 0 0" />
-      <mass
-        value="0.369742076927137" />
-      <inertia
-        ixx="0.00246788834863717"
-        ixy="4.99944210740992E-08"
-        ixz="-3.25489511678092E-08"
-        iyy="0.00211847372798997"
-        iyz="0.000668250395065579"
-        izz="0.000839231486986835" />
+        xyz="1.72360446946572E-06 -0.0572841318243815 0.203781479974732"
+        rpy="0 0 0" />
+      <mass
+        value="1.11383740307423" />
+      <inertia
+        ixx="0.00840848075882267"
+        ixy="1.16819985276106E-10"
+        ixz="3.20661375501498E-08"
+        iyy="0.0068932070989986"
+        iyz="0.00249453758997878"
+        izz="0.00249504881189781" />
     </inertial>
     <visual>
@@ -277,5 +277,5 @@
         name="">
         <color
-          rgba="0.501960784313725 0.501960784313725 0.501960784313725 1" />
+          rgba="0.752941176470588 0.752941176470588 0.752941176470588 1" />
       </material>
     </visual>
@@ -294,6 +294,6 @@
     type="revolute">
     <origin
-      xyz="0 0.061 0.101"
-      rpy="0 0 0" />
+      xyz="0 0 0"
+      rpy="1.5708 0 1.5708" />
     <parent
       link="elfin_link3" />
@@ -312,15 +312,15 @@
     <inertial>
       <origin
-        xyz="-1.43602737885348E-06 0.0400732712700223 0.0365459315107893"
-        rpy="0 0 0" />
-      <mass
-        value="0.810519795979025" />
-      <inertia
-        ixx="0.00228900919014725"
-        ixy="3.53045982931884E-08"
-        ixz="2.29268789681775E-08"
-        iyy="0.00188329109495946"
-        iyz="-0.000564395858742294"
-        izz="0.00101935359998985" />
+        xyz="3.18971281487254E-07 -0.0247904768102997 -0.00288553868007254"
+        rpy="0 0 0" />
+      <mass
+        value="0.932428626153683" />
+      <inertia
+        ixx="0.00225363150047226"
+        ixy="1.57057111903631E-08"
+        ixz="6.68352833152811E-08"
+        iyy="0.00123622421076959"
+        iyz="7.71608214306329E-05"
+        izz="0.00173913787162088" />
     </inertial>
     <visual>
@@ -335,5 +335,5 @@
         name="">
         <color
-          rgba="0.772549019607843 0.752941176470588 0.733333333333333 1" />
+          rgba="1 1 1 1" />
       </material>
     </visual>
@@ -352,6 +352,6 @@
     type="revolute">
     <origin
-      xyz="0 -0.056 0.223"
-      rpy="0 0 0" />
+      xyz="0 0 0.324"
+      rpy="-1.5708 0 0" />
     <parent
       link="elfin_link4" />
@@ -359,5 +359,5 @@
       link="elfin_link5" />
     <axis
-      xyz="0 1 0" />
+      xyz="0 0 1" />
     <limit
       lower="-2.56"
@@ -370,15 +370,15 @@
     <inertial>
       <origin
-        xyz="3.20814749367106E-05 -0.00725494085500073 0.0375620352744778"
-        rpy="0 0 0" />
-      <mass
-        value="0.11342880515576" />
-      <inertia
-        ixx="7.66530991301819E-05"
-        ixy="-1.83940471442645E-07"
-        ixz="-4.80914267075654E-08"
-        iyy="7.49230832326719E-05"
-        iyz="-2.34292724113658E-06"
-        izz="0.000127800839988254" />
+        xyz="1.4323826069585E-07 -0.00502093248893552 0.129189718099031"
+        rpy="0 0 0" />
+      <mass
+        value="0.288820351990399" />
+      <inertia
+        ixx="0.00021791903145322"
+        ixy="9.9472362909318E-10"
+        ixz="3.50877282174168E-11"
+        iyy="0.000175921298751184"
+        iyz="1.17498406450176E-06"
+        izz="0.000299410517394812" />
     </inertial>
     <visual>
@@ -393,5 +393,5 @@
         name="">
         <color
-          rgba="0.776470588235294 0.756862745098039 0.737254901960784 1" />
+          rgba="1 1 1 1" />
       </material>
     </visual>
@@ -410,6 +410,6 @@
     type="revolute">
     <origin
-      xyz="0 0.056 0.096"
-      rpy="0 0 0" />
+      xyz="0 0 0"
+      rpy="1.5708 0 0" />
     <parent
       link="elfin_link5" />
@@ -424,8 +424,12 @@
       velocity="1.57" />
   </joint>
-  <link name="elfin_end_link"/>
-  <joint name="elfin_end_joint" type="fixed">
-    <origin
-      xyz="0 0 0.059"
+  <link
+    name="elfin_end_link">
+  </link>
+  <joint
+    name="elfin_end_joint"
+    type="fixed">
+    <origin
+      xyz="0 0 0.155"
       rpy="0 0 0" />
     <parent
@@ -433,4 +437,6 @@
     <child
       link="elfin_end_link" />
+    <axis
+      xyz="0 0 0" />
   </joint>
   <link name="elfin_dummy_gripper"/>
