Commit message: update model
update model and urdf

File: elfin5_l/elfin5_l_ros2_gazebo/urdf/elfin5_l.urdf.xacro (robot description, xacro)
@@ -30,5 +30,5 @@
     <origin
       xyz="0 0 0"
-      rpy="0 0 1.5708" />
+      rpy="0 0 0" />
     <parent
       link="elfin_base_link" />
@@ -40,15 +40,15 @@
     <inertial>
       <origin
-        xyz="0.00022093 0.0013404 0.025529"
-        rpy="0 0 0" />
-      <mass
-        value="0.68795" />
-      <inertia
-        ixx="0.0012704"
-        ixy="6.1256E-06"
-        ixz="1.9788E-06"
-        iyy="0.0013413"
-        iyz="1.2007E-05"
-        izz="0.0022564" />
+        xyz="-0.00199130179727394 7.44168336203446E-06 0.0272977448147404"
+        rpy="0 0 0" />
+      <mass
+        value="0.546250568289568" />
+      <inertia
+        ixx="0.00118732326275469"
+        ixy="5.36844840925411E-07"
+        ixz="-2.09426769103823E-05"
+        iyy="0.00103230683074767"
+        iyz="-1.04918150299868E-07"
+        izz="0.00193030289476119" />
     </inertial>
     <visual>
@@ -63,5 +63,5 @@
         name="">
         <color
-          rgba="0.79216 0.81961 0.92941 1" />
+          rgba="0.792156862745098 0.819607843137255 0.933333333333333 1" />
       </material>
     </visual>
@@ -80,15 +80,15 @@
     <inertial>
       <origin
-        xyz="-0.021818 0.13889 0.000013458"
-        rpy="0 0 0" />
-      <mass
-        value="2.5856" />
-      <inertia
-        ixx="0.012636"
-        ixy="0.0034176"
-        ixz="-1.9559E-06"
-        iyy="0.0066118"
-        iyz="-1.7982E-06"
-        izz="0.014362" />
+        xyz="3.55428747498904E-05 -0.0238032507595431 -0.056664005378111"
+        rpy="0 0 0" />
+      <mass
+        value="1.71757344675846" />
+      <inertia
+        ixx="0.00313309686683817"
+        ixy="-6.81025650006338E-07"
+        ixz="-2.50470833748591E-06"
+        iyy="0.00372508389579096"
+        iyz="0.000325673248643593"
+        izz="0.00319411847606861" />
     </inertial>
     <visual>
@@ -103,5 +103,5 @@
         name="">
         <color
-          rgba="0.77255 0.75294 0.73333 1" />
+          rgba="0.792156862745098 0.819607843137255 0.933333333333333 1" />
       </material>
     </visual>
@@ -120,6 +120,6 @@
     type="revolute">
     <origin
-      xyz="0 0 0.03"
-      rpy="1.5708 0 0" />
+      xyz="0 0 0.22"
+      rpy="0 0 0" />
     <parent
       link="elfin_base" />
@@ -127,9 +127,9 @@
       link="elfin_link1" />
     <axis
-      xyz="0 1 0" />
+      xyz="0 0 1" />
     <limit
       lower="-3.14"
       upper="3.14"
-      effort="420"
+      effort="104"
       velocity="1.57" />
   </joint>
@@ -138,15 +138,15 @@
     <inertial>
       <origin
-        xyz="-0.032497 0.30341 -7.6521E-05"
-        rpy="0 0 0" />
-      <mass
-        value="1.208607" />
-      <inertia
-        ixx="0.02975970"
-        ixy="-0.00126441"
-        ixz="-0.00000024"
-        iyy="0.00168156"
-        iyz="-0.0000021"
-        izz="0.02944694" />
+        xyz="-8.02320899791198E-06 0.194762833402907 0.128888916941187"
+        rpy="0 0 0" />
+      <mass
+        value="1.10522962809227" />
+      <inertia
+        ixx="0.0225843178593198"
+        ixy="-7.27982747203185E-07"
+        ixz="-1.78485875318381E-07"
+        iyy="0.00152004282471311"
+        iyz="0.000623589021520354"
+        izz="0.0230428803086098" />
     </inertial>
     <visual>
@@ -161,5 +161,5 @@
         name="">
         <color
-          rgba="0.68627 0.68627 0.68627 1" />
+          rgba="0.792156862745098 0.819607843137255 0.933333333333333 1" />
       </material>
     </visual>
@@ -178,6 +178,6 @@
     type="revolute">
     <origin
-      xyz="-0.087 0.19 0"
-      rpy="0 0 0" />
+      xyz="0 0 0"
+      rpy="1.5708 0 0" />
     <parent
       link="elfin_link1" />
@@ -185,10 +185,10 @@
       link="elfin_link2" />
     <axis
-      xyz="-1 0 0" />
-    <limit
+      xyz="0 0 1" />
+     <limit
       lower="-2.35"
       upper="2.35"
-      effort="420"
-      velocity="1.57" />
+      effort="104"
+      velocity="1.27" />
   </joint>
   <link
@@ -196,15 +196,15 @@
     <inertial>
       <origin
-        xyz="0.067584 -0.041479 -1.1421E-05"
-        rpy="0 0 0" />
-      <mass
-        value="1.5324" />
-      <inertia
-        ixx="0.00514"
-        ixy="0.0014834"
-        ixz="-5.7782E-07"
-        iyy="0.0028926"
-        iyz="-3.0654E-07"
-        izz="0.0060883" />
+        xyz="0.0461694549854045 1.67843463302067E-05 -0.0210719533256843"
+        rpy="0 0 0" />
+      <mass
+        value="1.07590672952063" />
+      <inertia
+        ixx="0.00137807691049161"
+        ixy="-3.57302576480749E-07"
+        ixz="-0.00013179565326652"
+        iyy="0.00135308160804782"
+        iyz="9.02259193989242E-07"
+        izz="0.00154416453671479" />
     </inertial>
     <visual>
@@ -219,5 +219,5 @@
         name="">
         <color
-          rgba="0.86667 0.86667 0.8902 1" />
+          rgba="0.792156862745098 0.819607843137255 0.933333333333333 1" />
       </material>
     </visual>
@@ -237,5 +237,5 @@
     <origin
       xyz="0 0.455 0"
-      rpy="-3.1416 0 0" />
+      rpy="-3.1416 0 1.5708" />
     <parent
       link="elfin_link2" />
@@ -243,179 +243,63 @@
       link="elfin_link3" />
     <axis
-      xyz="1 0 0" />
+      xyz="0 0 1" />
     <limit
       lower="-2.61"
       upper="2.61"
-      effort="200"
-      velocity="1.57" />
-  </joint>
-  <link
-    name="elfin_link4">
-    <inertial>
-      <origin
-        xyz="-0.017434 -0.33294 -0.00015134"
-        rpy="0 0 0" />
-      <mass
-        value="0.5" />
-      <inertia
-        ixx="0.00542441"
-        ixy="0.0020749"
-        ixz="1.0501E-05"
-        iyy="0.014338"
-        iyz="-0.00041574"
-        izz="0.00607489" />
-    </inertial>
-    <visual>
-      <origin
-        xyz="0 0 0"
-        rpy="0 0 0" />
-      <geometry>
-        <mesh
-          filename="file://$(find elfin_description)/meshes/elfin5_l/elfin_link4.STL" />
-      </geometry>
-      <material
-        name="">
-        <color
-          rgba="0.68627 0.68627 0.68627 1" />
-      </material>
-    </visual>
-    <collision>
-      <origin
-        xyz="0 0 0"
-        rpy="0 0 0" />
-      <geometry>
-        <mesh
-          filename="file://$(find elfin_description)/meshes/elfin5_l/elfin_link4.STL" />
-      </geometry>
-    </collision>
-  </link>
-  <joint
-    name="elfin_joint4"
-    type="revolute">
-    <origin
-      xyz="0.087 -0.1255 0"
-      rpy="3.1416 0 0" />
-    <parent
-      link="elfin_link3" />
-    <child
-      link="elfin_link4" />
-    <axis
-      xyz="0 1 0" />
-    <limit
-      lower="-3.14"
-      upper="3.14"
-      effort="200"
-      velocity="1.57" />
-  </joint>
-  <link
-    name="elfin_link5">
-    <inertial>
-      <origin
-        xyz="-0.015972 -0.036591 1.4235E-06"
-        rpy="0 0 0" />
-      <mass
-        value="0.81192" />
-      <inertia
-        ixx="0.0018901"
-        ixy="0.00056728"
-        ixz="-4.2025E-08"
-        iyy="0.0010231"
-        iyz="5.0791E-09"
-        izz="0.002299" />
-    </inertial>
-    <visual>
-      <origin
-        xyz="0 0 0"
-        rpy="0 0 0" />
-      <geometry>
-        <mesh
-          filename="file://$(find elfin_description)/meshes/elfin5_l/elfin_link5.STL" />
-      </geometry>
-      <material
-        name="">
-        <color
-          rgba="0.79216 0.81961 0.93333 1" />
-      </material>
-    </visual>
-    <collision>
-      <origin
-        xyz="0 0 0"
-        rpy="0 0 0" />
-      <geometry>
-        <mesh
-          filename="file://$(find elfin_description)/meshes/elfin5_l/elfin_link5.STL" />
-      </geometry>
-    </collision>
-  </link>
-  <joint
-    name="elfin_joint5"
-    type="revolute">
-    <origin
-      xyz="0 0.3695 0"
-      rpy="-3.1416 0 0" />
-    <parent
-      link="elfin_link4" />
-    <child
-      link="elfin_link5" />
-    <axis
-      xyz="1 0 0" />
-    <limit
-      lower="-2.56"
-      upper="2.56"
       effort="69"
       velocity="1.57" />
   </joint>
   <link
-    name="elfin_link6">
-    <inertial>
-      <origin
-        xyz="-0.0072549 0.027062 3.208E-05"
-        rpy="0 0 0" />
-      <mass
-        value="0.11343" />
-      <inertia
-        ixx="7.4923E-05"
-        ixy="-2.3429E-06"
-        ixz="-1.8394E-07"
-        iyy="0.0001278"
-        iyz="-4.8092E-08"
-        izz="7.6653E-05" />
-    </inertial>
-    <visual>
-      <origin
-        xyz="0 0 0"
-        rpy="0 0 0" />
-      <geometry>
-        <mesh
-          filename="file://$(find elfin_description)/meshes/elfin5_l/elfin_link6.STL" />
-      </geometry>
-      <material
-        name="">
-        <color
-          rgba="0.77647 0.75686 0.73725 1" />
-      </material>
-    </visual>
-    <collision>
-      <origin
-        xyz="0 0 0"
-        rpy="0 0 0" />
-      <geometry>
-        <mesh
-          filename="file://$(find elfin_description)/meshes/elfin5_l/elfin_link6.STL" />
-      </geometry>
-    </collision>
-  </link>
-  <joint
-    name="elfin_joint6"
-    type="revolute">
-    <origin
-      xyz="0 -0.1065 0"
-      rpy="3.1416 0 0" />
-    <parent
-      link="elfin_link5" />
-    <child
-      link="elfin_link6" />
-    <axis
-      xyz="0 1 0" />
+    name="elfin_link4">
+    <inertial>
+      <origin
+        xyz="-2.52415186551188E-05 -0.0426485662035081 0.296130346848396"
+        rpy="0 0 0" />
+      <mass
+        value="0.773486357600959" />
+      <inertia
+        ixx="0.0065953698905962"
+        ixy="-7.26135070513294E-07"
+        ixz="2.7130632453124E-06"
+        iyy="0.00593057161737003"
+        iyz="0.00162601275838063"
+        izz="0.00175532385127571" />
+    </inertial>
+    <visual>
+      <origin
+        xyz="0 0 0"
+        rpy="0 0 0" />
+      <geometry>
+        <mesh
+          filename="file://$(find elfin_description)/meshes/elfin5_l/elfin_link4.STL" />
+      </geometry>
+      <material
+        name="">
+        <color
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